File: Hardware/Reverse Polarity Protection.kicad_pcb (KiCad board)
At the start: 2 copper layers, 66.9 x 42.1 mm, 14 parts, among them CON1 VIN, CON2 GND, CON3 VOUT, CON4 GND, J1 Screw_Terminal_01x02, Q1 SUM40N10-30-E3, U1 LM5050-1

Commit message: KiCad 8.0
Routing:
- net GND: track 190.6 -> 254.9 mm
- net /VOUT: track 98.1 -> 140.4 mm
- net /VIN: track 93.7 -> 126.4 mm
- net /Vs: track 9.23 -> 9.97 mm
