File: Hardware/ReversePolarityProtection.kicad_pcb (KiCad board)
At the start: 2 copper layers, 66.9 x 42.1 mm, 14 parts, among them CON1 VIN, CON2 GND, CON3 VOUT, CON4 GND, J1 Screw_Terminal_01x02, Q1 SUM40N10-30-E3, U1 LM5050-1

Commit message: Fix missing D2
Parts:
- added D2: SS16T3G, Diode_SMD:D_SMA-SMB_Universal_Handsoldering, F.Cu at (67.8, 116.3)
- moved D1 6.73 mm to (74.0, 112.5)
- moved C3 5.28 mm to (86.3, 105.8)
- moved R1 5.28 mm to (89.5, 106.8)
- moved R2 5.28 mm to (89.5, 104.5)
- moved U1 5.28 mm to (82.0, 106.5)
- moved J1 5.28 mm to (84.0, 100.9)
- moved D3 1.78 mm to (112.3, 116.0)
- moved Q1 1.78 mm to (87.2, 116.0)
- moved C2 1.78 mm to (101.6, 116.0)
- renumbered D2 to D3
Connections:
- D1 pad 2: GND -> Net-(D1-A)
Routing:
- net /VOUT: track 140.4 -> 122.8 mm, vias 0 -> 39
- net /VIN: track 126.4 -> 113.4 mm, vias 0 -> 27
- net Net-(D1-A): track 0.00 -> 7.05 mm
- net /Gate_Drive: track 8.51 -> 5.95 mm
- net /Vs: track 9.97 -> 9.11 mm
- net GND: track 254.9 -> 254.0 mm, vias 2 -> 72
- added copper zone on B.Cu, net /VIN
- added copper zone on B.Cu, net /VOUT
Other:
- board text added: "{ "ViaStitching": "0.2", "stitch_zone_0": { "HSpacing": "1", "VSpacing": "1", "Clearance": "0", "Randomize": true }, "stitch_zone_1": { "HSpacing": "1", "VSpacing": "1", "Clearance": "0", "Randomize": true } }"
